File: ecad/UPS/Charger.kicad_sch (KiCad schematic)
At the start: 0 parts

Commit message: Did some routing, need to figure out how to route to BQ while appeasing DRC
Parts:
- added B1, B2, B3, B4: 1121, UPS:1121_KEY, symbol UPS:1121
- added C1, C2: 100pF, Capacitor_SMD:C_0603_1608Metric, symbol Device:C
- added C13, C15: 33nF, Capacitor_SMD:C_0603_1608Metric, symbol Device:C
- added C14, C45: 10nF, Capacitor_SMD:C_0603_1608Metric, symbol Device:C
- added C16: 47nF, Capacitor_SMD:C_0603_1608Metric, symbol Device:C
- added C17: 47 nF, Capacitor_SMD:C_0603_1608Metric, symbol Device:C
- added C27: 1uF, Capacitor_SMD:C_0603_1608Metric, symbol Device:C
- added C28: 15pF, Capacitor_SMD:C_0603_1608Metric, symbol Device:C
- added C29: 33pF, Capacitor_SMD:C_0603_1608Metric, symbol Device:C
- added C30: 1200 pF, Capacitor_SMD:C_0603_1608Metric, symbol Device:C
- added C31: 3.3nF, Capacitor_SMD:C_0603_1608Metric, symbol Device:C
- added C32: .1µF, Capacitor_SMD:C_0603_1608Metric, symbol Device:C
- added C33, C37, C39, C40, C41, C42, C43, C44, C51, C52, C53, C54, C55, C56, C57: 10µF, Capacitor_SMD:C_0603_1608Metric, symbol Device:C
- added C34, C38: 1µF, Capacitor_SMD:C_0603_1608Metric, symbol Device:C
- added C46: 1 nF, Capacitor_SMD:C_0603_1608Metric, symbol Device:C
- added C47, C48: 22µF, Capacitor_SMD:C_1206_3216Metric, symbol Device:C
- added C58: 2.2µF, Capacitor_SMD:C_0603_1608Metric, symbol Device:C
- added D7: D_Zener, Diode_SMD:D_SMB_Handsoldering, symbol Device:D_Zener
- added J1: Barrel_Jack, Connector_BarrelJack:BarrelJack_Horizontal, symbol Connector:Barrel_Jack
- added J2: Conn_01x02_Socket, Connector_AMASS:AMASS_XT60-F_1x02_P7.20mm_Vertical, symbol Connector:Conn_01x02_Socket
- added L1: 2.2µH, Inductor_SMD:L_Vishay_IHLP-4040, symbol Device:L
- added Q1, Q5, Q6, Q7: CSD18540Q5B, UPS:TRANS_CSD18540Q5B, symbol UPS:CSD18540Q5B
- added Q2: Q_PMOS_DGS, UPS:FDS6681Z_OSI-M, symbol UPS:FDS6681Z
- added Q4: Q_PMOS_DGS, UPS:FDS6681Z_OSI, symbol UPS:FDS6681Z
- added R1: 140k, Resistor_SMD:R_0805_2012Metric, symbol Device:R
- added R11, R17: .01, Resistor_SMD:R_2512_6332Metric, symbol Device:R
- added R12: 2.2, Resistor_SMD:R_0805_2012Metric, symbol Device:R
- added R13: 16.9k, Resistor_SMD:R_0805_2012Metric, symbol Device:R
- added R14, R2: 10k, Resistor_SMD:R_0805_2012Metric, symbol Device:R
- added R24, R28, R34: 68.1k, Resistor_SMD:R_0805_2012Metric_Pad1.20x1.40mm_HandSolder, symbol Device:R
- added R25: 60k, Resistor_SMD:R_0805_2012Metric, symbol Device:R
- added R26: 20k, Resistor_SMD:R_0805_2012Metric, symbol Device:R
- added R27, R4: 100k, Resistor_SMD:R_0805_2012Metric, symbol Device:R
- added R3: 56k, Resistor_SMD:R_0805_2012Metric, symbol Device:R
- added R5: 10, Resistor_SMD:R_0805_2012Metric, symbol Device:R
- added TH2, TH3, TH4: B57471V2104J062, Resistor_SMD:R_0805_2012Metric_Pad1.20x1.40mm_HandSolder, symbol Device:Thermistor_NTC
- added U1: BQ25730RSNR, UPS:RSN0032B-IPC_A, symbol UPS:BQ25730RSNR
Connections:
- new net: B1.2, B2.2, B3.2, B4.2, C32.1, C33.1, C37.1, J2.1 (Pin_1), R17.2, U1.19 (SRN)
- new net: C13.1, C14.2, C45.1, C46.1, Q7.5_6_7_8, R11.1, U1.2 (ACN)
- new net: D7.2 (A), Q2.4, R27.2
- new net: J1.1, Q2.5, Q2.6, Q2.7, Q2.8
- new net: R2.1, U1.10 (PSYS)
- new net: C32.2, C34.1, Q4.5, Q4.6, Q4.7, Q4.8, R17.1, U1.20 (SRP)
- new net: C27.2, R12.1
- new net: R25.2, R26.1, U1.18 (CELL_BATPRESZ)
- new net: C1.1, U1.9 (IBAT)
- new net: Q6.4, U1.29 (LODRV1)
- new net: Q5.4, U1.26 (LODRV2)
- new net: C17.2, L1.2, Q1.1, Q1.2, Q1.3, Q5.5_6_7_8, U1.23 (SW2)
- new net: C30.2, R14.2
- new net: C31.2, R13.2
- new net: Q1.4, U1.24 (HIDRV2)
- new net: C2.1, R1.1, U1.8 (IADPT)
- new net: Q4.4, U1.21 (BATDRV_N)
- new net +3.3V: R24.1, R28.1, R34.1
- new net BTST1: C16.1, U1.30 (BTST1)
- new net BTST2: C17.1, U1.25 (BTST2)
- new net CMPIN: U1.14 (CMPIN)
- new net COMP1: C29.2, R13.1, U1.16 (COMP1)
- new net COMP2: C28.2, R14.1, U1.17 (COMP2)
- new net GND: B1.1, B2.1, B3.1, B4.1, C1.2, C13.2, C15.1, C2.2, C27.1, C28.1, C29.1, C30.1, C31.1, C33.2, C34.2, C37.2, C38.2, C39.2, C40.2, C41.2, C42.2, C43.2, C44.2, C45.2, C46.2, C47.2, C48.2, C51.2, C52.2, C53.2, C54.2, C55.2, C56.2, C57.2, C58.2, J1.2, J2.2 (Pin_2), Q5.1, Q5.2, Q5.3, Q6.1, Q6.2, Q6.3, Q7.4, R1.2, R2.2, R26.2, R27.1, R3.2, TH2.2, TH3.2, TH4.2, U1.27 (PGND), U1.31 (HIDRV1), U1.33 (Thermal_Pad)
- new net ILIM_HIZ: R3.1, R4.2, U1.6 (ILIM_HIZ)
- new net OTG/VAP: U1.5 (OTG_VAP)
- new net PMOS_IN_GATE: C14.1, C15.2, C39.1, C40.1, C41.1, C42.1, C43.1, C44.1, D7.1 (K), Q2.1, Q2.2, Q2.3, R11.2, R12.2, U1.1 (VBUS), U1.3 (ACP)
- new net PMOS_OUT_GATE: C47.1, C48.1, C51.1, C52.1, C53.1, C54.1, C55.1, C56.1, C57.1, Q1.5_6_7_8, Q4.1, Q4.2, Q4.3, U1.22 (VSYS)
- new net PROCHOT_N: U1.11 (PROCHOT_N)
- new net REGN: C58.1, R5.1, U1.28 (REGN)
- new net SW1: C16.2, L1.1, Q6.5_6_7_8, Q7.1, Q7.2, Q7.3, U1.32 (SW1)
- new net VDDA: C38.1, R25.1, R4.1, R5.2, U1.7 (VDDA)
- new net bat_th1: R24.2, TH2.1
- new net bat_th2: R28.2, TH3.1
- new net bat_th3: R34.2, TH4.1
- new net chrg_ok: U1.4 (CHRG_OK)
- new net cmp_out: U1.15 (CMPOUT)
- new net i2c_scl: U1.13 (SCL)
- new net i2c_sda: U1.12 (SDA)
Other:
- company: (none) -> MTU Open Source Hardware Enterprise
- title: (none) -> Charger

Commit message: Ty's changes from this morning
Parts:
- removed C27: 1uF, Capacitor_SMD:C_0603_1608Metric, symbol Device:C
- removed R12: 2.2, Resistor_SMD:R_0805_2012Metric, symbol Device:R
- U1: footprint UPS:RSN0032B-IPC_A -> UPS:RSN0032B-IPC_C
Connections:
- net GND: no longer C1.2, C2.2, C28.1, C29.1, C30.1, C31.1, C38.2, R1.2, R2.2, R26.2, R3.2
- new net GNDA: C1.2, C2.2, C28.1, C29.1, C30.1, C31.1, C38.2, R1.2, R2.2, R26.2, R3.2
