File: ecad/UPS/UPS.kicad_pcb (KiCad board)
At the start: 4 copper layers, 177.8 x 139.7 mm, 160 parts, among them J1 Barrel_Jack, J2 Conn_01x02_Socket, J3 USB_C_Receptacle_USB2.0_16P, J4 PROG, Q1 CSD18540Q5B, Q2 Q_PMOS_DGS, Q3 IRLR7843TRPBF, Q4 Q_PMOS_DGS, Q5 CSD18540Q5B, Q6 CSD18540Q5B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

Commit message: Ty's changes from this morning
Parts:
- removed C27: 1uF, Capacitor_SMD:C_0603_1608Metric
- removed R12: 2.2, Resistor_SMD:R_0805_2012Metric
- U1: footprint UPS:RSN0032B-IPC_A -> UPS:RSN0032B-IPC_C
- moved C45 21.0 mm to (92.5, 51.7), turned to -90 degrees
- moved C46 18.3 mm to (107.2, 58.5)
- moved C13 16.9 mm to (101.3, 58.5)
- moved C33 14.0 mm to (123.5, 65.2), turned to -90 degrees
- moved C15 13.3 mm to (102.5, 67.2), turned to 90 degrees
- moved C14 13.0 mm to (103.8, 64.0)
- moved C28 8.41 mm to (111.2, 72.0)
- moved C51 2.55 mm to (149.3, 45.6)
- moved C52 2.55 mm to (149.3, 43.5)
- moved C53 2.55 mm to (149.3, 57.7)
- moved C54 2.55 mm to (149.3, 55.2)
- moved C55 2.55 mm to (149.3, 52.6)
- moved C56 2.55 mm to (149.3, 50.1)
- moved C57 2.55 mm to (149.3, 47.6)
- moved Q1 2.55 mm to (143.0, 45.5)
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Connections:
- C1 pad 2: PGND -> GNDA
- C2 pad 2: PGND -> GNDA
- C28 pad 1: PGND -> GNDA
- C29 pad 1: PGND -> GNDA
- C30 pad 1: PGND -> GNDA
- C31 pad 1: PGND -> GNDA
- C38 pad 2: PGND -> GNDA
- R1 pad 2: PGND -> GNDA
- R2 pad 2: PGND -> GNDA
- R26 pad 2: PGND -> GNDA
- R3 pad 2: PGND -> GNDA
Routing:
- net PMOS_IN_GATE: track 51.1 -> 131.9 mm
- net PMOS_OUT_GATE: track 0.00 -> 25.2 mm
- net Net-(U1-ACN): track 20.3 -> 42.0 mm
- net PGND: track 84.8 -> 101.7 mm, vias 87 -> 99
- net Net-(U1-SW2): track 29.9 -> 16.6 mm
- net BTST2: track 0.00 -> 8.16 mm
- net Net-(U1-SRP): track 0.00 -> 7.70 mm
- net (no net): track 0.00 -> 1.00 mm
- net GNDA: track 0.00 -> 0.09 mm, vias 0 -> 3
- removed copper zone on F.Cu, net PMOS_OUT_GATE
